File: hw/pico-audio-visualizer/pico-audio-visualizer.kicad_sch (KiCad schematic)
At the start: 0 parts

Commit message: WIP
Parts:
- added C1, C3, C6: 100nF, symbol Device:C
- added C2, C4, C5: 1uF, symbol Device:C
- added C7: 6.8n, symbol Device:C
- added C8: 1u, symbol Device:C
- added J1: Audio_In, symbol Connector:Conn_01x03_Pin
- added J2: Audio_Out, symbol Connector:Conn_01x03_Pin
- added R1, R3: 10k, symbol Device:R
- added R10, R9: 1k, symbol Device:R
- added R2, R4: 220, symbol Device:R
- added R5, R6: 100, symbol Device:R
- added R7: 100k, symbol Device:R
- added R8: 510, symbol Device:R
- added RV1: 1k, symbol Device:R_Potentiometer
- added RV2: 200k, symbol Device:R_Potentiometer
- added U1, U3: CD4051B, Package_DIP:DIP-16_W7.62mm_Socket, symbol Analog_Switch:CD4051B
- added U2: Pico, MCU_RaspberryPi_and_Boards:RPi_Pico_SMD_TH, symbol MCU_RaspberryPi_and_Boards:Pico
- added U4: TL431P, Package_DIP:DIP-8_W7.62mm, symbol Reference_Voltage:TL431P
Connections:
- new net: J1.1 (Pin_1), J2.1 (Pin_1), R9.1
- new net: J1.2 (Pin_2), J2.2 (Pin_2), R10.1
- new net: C7.1, C8.1, R8.2
- new net: R5.2, U3.1 (X4), U3.12 (X3), U3.15 (X2), U3.2 (X6), U3.4 (X7), U3.5 (X5)
- new net: U2.25 (GPIO19), U3.10 (B)
- new net: U2.24 (GPIO18), U3.11 (A)
- new net: R4.1, U3.3 (X)
- new net: R3.1, U2.21 (GPIO16), U3.6 (INH)
- new net: R6.1, U3.9 (C)
- new net: R10.2, R7.1, R8.1, R9.2
- new net: RV1.2, U4.8 (REF)
- new net: U1.10 (B), U2.15 (GPIO11)
- new net: U1.11 (A), U2.16 (GPIO12)
- new net: R2.1, U1.3 (X)
- new net: R1.1, U1.6 (INH), U2.20 (GPIO15)
- new net: U1.9 (C), U2.14 (GPIO10)
- new net +1.65V: C8.2, RV2.2, U2.31 (GPIO26_ADC0)
- new net +3.3V: RV2.1, U2.35 (ADC_VREF), U4.1 (K)
- new net +5V: C1.2, C2.1, C3.2, C4.1, C5.2, C6.2, R1.2, R2.2, R3.2, R4.2, RV1.1, U1.16 (VDD), U2.40 (VBUS), U3.16 (VDD)
- new net GNDA: C7.2, J1.3 (Pin_3), J2.3 (Pin_3), R7.2, U2.33 (AGND)
- new net GNDPWR: C1.1, C2.2, C3.1, C4.2, C5.1, C6.1, R5.1, R6.2, RV2.3, U1.7 (VEE), U1.8 (VSS), U2.13 (GND), U2.18 (GND), U2.23 (GND), U2.28 (GND), U2.3 (GND), U2.38 (GND), U2.8 (GND), U3.7 (VEE), U3.8 (VSS), U4.6 (A)
- new net LED0: U2.12 (GPIO9)
- new net LED1: U2.11 (GPIO8)
- new net LED2: U2.10 (GPIO7)
- new net LED3: U2.9 (GPIO6)
- new net LED4: U2.7 (GPIO5)
- new net LED5: U2.6 (GPIO4)
- new net LED6: U2.5 (GPIO3)
- new net LED7: U2.4 (GPIO2)
- new net Sink0: U1.13 (X0)
- new net Sink1: U1.14 (X1)
- new net Sink2: U1.15 (X2)
- new net Sink3: U1.12 (X3)
- new net Sink4: U1.1 (X4)
- new net Sink5: U1.5 (X5)
- new net Sink6: U1.2 (X6)
- new net Sink7: U1.4 (X7)
- new net Sink8: U3.13 (X0)
- new net Sink9: U3.14 (X1)
Other:
- note added: "ADC VREF and input biasing voltage"
- note added: "Input signal The stereo signal is passed through the Audio Out connector before it is mixed to mono"
